Commit message: add matrix

File: js/example/dev-bundle/gp180/urdf/gp180.urdf (robot description, URDF)
Before this commit: robot gp180, 7 links, 6 joints
Joints:
- removed joint join4
- added joint joint4: type revolute, parent Empty_Link_3, child Empty_Link_4, origin xyz=1.033 -0.3 -0.0415 rpy=3.1416 1.5708 0, axis 0 0 -1, limit lower=-6.283 upper=6.283 effort=1000 velocity=3.18
